File: Funktionsgenerator_lm324/Funktionsgenerator.kicad_sch (KiCad schematic)
At the start: 38 parts, among them J1 Conn_01x02_Socket, J10 to Freq. select, J11 Conn_01x03_Pin, J12 Conn_01x03_Socket, J2 Freq. select, J3 Conn_01x03_Socket, J4 Screw_Terminal_01x02, J5 to ampl. adj., J6 freq adj., J9 to freq adj.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

Commit message: Add files via upload
Parts:
- removed J5: to ampl. adj., symbol Connector:Conn_01x02_Pin
- added C11: C, symbol Device:C
- added J5: to ampl. adj, symbol Connector:Conn_01x03_Pin
- added J7: ampl. adj, symbol Connector:Conn_01x03_Socket
- R6: value 330# -> 1k
- R7: value 330 -> 500
Connections:
- net GND: now also R7.2, J7.1 (Pin_1); no longer R6.1
- net at RV1.1: now also J5.1 (Pin_1)
- net at RV1.2: now also J5.3 (Pin_3)
- net at RV1.3: now also J5.2 (Pin_2)
- net at R6.2, R7.1: now also U2.3 (+), C11.2; no longer U2.13 (-)
- net at C9.2, U2.14: now also J7.3 (Pin_3); no longer R7.2
- net at U2.8, U2.9 (-): now also C11.1; no longer U2.3 (+)
- new net: J7.2 (Pin_2), U2.13 (-)
- new net +5V: R6.1
Other:
- moved on the sheet: C9, R, R3, R4, R5, U2A, U2B, U2D
